File: DuePrint3 KiCad Project/DuePrint3.kicad_sch (KiCad schematic)
At the start: 49 parts, among them J1 MF3.0-2x12-430452412, J10 MF3.0-1x2-436500215, J11 2.54Header-1x2-M, J12 2.54Header-1x2-M, J13 EHT-125-01-S-D, J14 EHT-110-01-S-D, J15 EHT-125-01-S-D, J2 2.54Header-1x16-F, J3 2.54Header-1x16-F, J4 6P2C, J5 6P2C, J6 2.54Header-1x3-M, J7 MF3.0-1x2-436500215, J8 MF3.0-1x8-436500815, J9 MF3.0-2x9-430451812, U1 SN74AHCT125DR

Commit message: v2.2.0 initial release
Primarily focused on KiCad files, configuration files, build instructions.
Parts:
- removed D1: 100v 1A, Diode_SMD:D_SMF, symbol Device:D_Schottky
- removed H4: MountingHole_Pad, Stratasys Adapter:MountingHole_4.00mm_Pad, symbol Mechanical:MountingHole_Pad
- removed J1: MF3.0-2x12-430452412, Connector_Molex:Molex_Micro-Fit_3.0_43045-2412_2x12_P3.00mm_Vertical, symbol Connector_Generic:Conn_02x12_Top_Bottom
- removed J11, J12: 2.54Header-1x2-M, Connector_PinHeader_2.54mm:PinHeader_1x02_P2.54mm_Vertical, symbol Connector_Generic:Conn_01x02
- removed J2, J3: 2.54Header-1x16-F, Connector_PinSocket_2.54mm:PinSocket_1x16_P2.54mm_Vertical, symbol Connector_Generic:Conn_01x16
- removed J8: MF3.0-1x8-436500815, Connector_Molex:Molex_Micro-Fit_3.0_43650-0815_1x08_P3.00mm_Vertical, symbol Connector_Generic:Conn_01x08
- removed J9: MF3.0-2x9-430451812, Connector_Molex:Molex_Micro-Fit_3.0_43045-1812_2x09_P3.00mm_Vertical, symbol Connector_Generic:Conn_02x09_Top_Bottom
- removed R10, R12, R16, R19: 3740, Resistor_SMD:R_0805_2012Metric_Pad1.20x1.40mm_HandSolder, symbol Device:R
- removed R11, R13, R15, R18: 31.6K, Resistor_SMD:R_0805_2012Metric_Pad1.20x1.40mm_HandSolder, symbol Device:R
- removed R24: 10k, Resistor_SMD:R_0805_2012Metric_Pad1.20x1.40mm_HandSolder, symbol Device:R
- added C2: 0.1 µF, Capacitor_SMD:C_0805_2012Metric_Pad1.18x1.45mm_HandSolder, symbol Device:C
- added C3: 10n 25V, Capacitor_SMD:C_0805_2012Metric_Pad1.18x1.45mm_HandSolder, symbol Device:C
- added J14: Conn_02x07_Top_Bottom, Connector_JST:JST_PHD_B14B-PHDSS_2x07_P2.00mm_Vertical, symbol Connector_Generic:Conn_02x07_Odd_Even
- added J16: Conn_02x15_Odd_Even, Connector_JST:JST_PHD_B30B-PHDSS_2x15_P2.00mm_Vertical, symbol Connector_Generic:Conn_02x15_Odd_Even
- added J6: Conn_01x02, Connector_PinHeader_2.54mm:PinHeader_2x01_P2.54mm_Vertical, symbol Connector_Generic:Conn_01x02
- added J8: MF3.0-1x2-436500215, Connector_Molex:Molex_Micro-Fit_3.0_43650-0215_1x02_P3.00mm_Vertical, symbol Connector_Generic:Conn_01x02
- added R17: 10k, Resistor_SMD:R_0805_2012Metric_Pad1.20x1.40mm_HandSolder, symbol Device:R
- added U2: SN74AHCT125DR, Package_SO:SOIC-14_3.9x8.7mm_P1.27mm, symbol SN74AHCT125DR:SN74AHCT125DR
- added U3: BLACKPILL, DuePrint3-Lib:STM32 BLACKPILL, symbol DuePrint3:STM32F411_BLACKPILL
- added U4: SAMMY-C21, DuePrint3-Lib:SAMMY-C21, symbol DuePrint3:SAMMY-C21
- J11: renamed from J4; footprint Connector_RJ:RJ12_Amphenol_54601-x06_Horizontal -> DuePrint3-Lib:BEL_SS-6466S-A-PG1
- J12: renamed from J5; footprint Connector_RJ:RJ12_Amphenol_54601-x06_Horizontal -> DuePrint3-Lib:BEL_SS-6466S-A-PG1
- R14: value 3740 -> 10k
- R9: value 31.6K -> 100K
- U1: footprint PCM_Package_SO_AKL:SOIC-14_3.9x8.7mm_P1.27mm -> Package_SO:SOIC-14_3.9x8.7mm_P1.27mm
- renumbered H3 to H2, H5 to H3, H2 to H4, H6 to H5, J14 to J1, J6 to J13, J13 to J2, J7 to J3, J10 to J4, J15 to J5, R8 to R1, R22 to R10, R23 to R11, R20 to R12, R21 to R13, R25 to R15, R17 to R16, R7 to R2, R1 to R4, R6 to R5, R4 to R6, R2 to R7, R5 to R8
Connections:
- net GECKO ERROR is gone; now on net Print Head Support Toggle SW: R13.1
- net VD EXTRUDER MODEL HEATER ENABLE is gone; now on an unnamed net: R9.1
- net +12V: now also J14.13 (Pin_13)
- net +5V: now also R14.1, C2.1, J14.9 (Pin_9), J16.27 (Pin_27), J8.2 (Pin_2), R17.1, U2.14 (VCC), U3.18 (5V), U3.21 (5V), U4.15 (V33), U4.17 (VCC); no longer J5.16 (Pin_16), U1.12 (4A), U1.13 (4~{OE})
- net ARMATURE NEGATIVE: now also U3.10 (PA15)
- net ARMATURE POSITIVE: now also U3.11 (PB03)
- net CAN0H: now also U4.32 (CAN0_H)
- net CAN0L: now also U4.31 (CAN0_L)
- net CHAMBER HEATER ENABLE: now also U1.11 (4Y); no longer R1.1, R2.2
- net CHAMBER TEMP ALARM: now also R10.2, U4.8 (PA07)
- net CHAMBER TEMP THERM: now also R8.2; no longer R5.2
- net DIR: now also U3.33 (PA02), U4.11 (PA10)
- net DOOR SOLENOID ENABLE: now also U2.11 (4Y); no longer U1.3 (1Y)
- net DOOR SWITCH: now also R12.1, U4.6 (PA05); no longer R11.2
- net ENCODER CH A: now also U3.29 (PA06)
- net ENCODER CH B: now also U3.30 (PA05)
- net GND: now also J2.12 (Pin_12), J2.6 (Pin_6), R9.2, C2.2, C3.2, J14.1 (Pin_1), J14.11 (Pin_11), J16.29 (Pin_29), J16.30 (Pin_30), J6.2 (Pin_2), J8.1 (Pin_1), U2.7 (GND), U3.19 (GND), U3.22 (GND), U4.16 (GND); no longer J5.24 (Pin_24), J5.26 (Pin_26), R14.2, U1.1 (1~{OE}), U1.10 (3~{OE}), U1.4 (2~{OE})
- net HEAD THERMOSTAT STATUS: now also R11.2, U4.7 (PA06); no longer R12.1
- net LED Lights Enable: now also U4.20 (PA24); no longer U1.6 (2Y)
- net LS DOOR SOLENOID ENABLE: now also J16.16 (Pin_16), U2.12 (4A); no longer U1.2 (1A)
- net MOTOR ENABLE: now also U1.8 (3Y)
- net PRINT BED TOUCH PR LIM SW: now also J16.7 (Pin_7)
- net PRINT HEAD TEMP ALARM: now also J16.23 (Pin_23)
- net Print Head Model Toggle SW: now also R15.2, U4.3 (PB08)
- net Print Head Support Toggle SW: now also U4.5 (PA04); no longer R10.2
- net STEP: now also U3.34 (PA01), U4.12 (PA11)
- net T0: now also R6.2, R8.1, J16.18 (Pin_18); no longer R3.1, R3.2, R5.1
- net T1: now also R3.2, R5.1, J16.26 (Pin_26); no longer R6.2, R8.1
- net T2: now also J16.22 (Pin_22)
- net X-AXIS HOME LIM SW: now also J16.15 (Pin_15)
- net X-Axis End of Travel Lim SW: now also J16.13 (Pin_13)
- net Y-AXIS HOME LIM SW: now also J16.17 (Pin_17)
- net Y-Axis End of Travel Lim SW: now also J16.11 (Pin_11)
- net Z-AXIS HOME LIM SW: now also J16.19 (Pin_19)
- net Z-Axis End of Travel Lim SW: now also J16.9 (Pin_9)
- net POWER ON: now reaches J5.21 (Pin_21)
- net POWER ON: now also U1.6 (2Y)
- net POWER I/O: now reaches J5.23 (Pin_23)
- net POWER I/O: now also J16.21 (Pin_21)
- net at J12.SH: now also J11.SH, C3.1
- net EMHE PWM renamed EXTRUDER MODEL HEATER ENABLE
- net EXTRUDER MODEL HEATER ENABLE: now also U2.8 (3Y); no longer R9.2
- net ESHE PWM renamed EXTRUDER SUPPORT HEATER ENABLE
- net EXTRUDER SUPPORT HEATER ENABLE: now also U2.6 (2Y)
- net FD1: no longer names the net of J1.2 (Pin_2)
- net FD2: no longer names the net of J1.3 (Pin_3)
- net LS GECKO RESET renamed LS MOTOR ENABLE
- net LS MOTOR ENABLE: now also J16.6 (Pin_6)
- net LS LED Lights Enable renamed LS POWER ON
- net LS POWER ON: now also J16.4 (Pin_4)
- net PBTPE PWM renamed PRINT BED TOUCH PR PWR EN
- net PRINT BED TOUCH PR PWR EN: now also U4.19 (PA25); no longer R14.1
- net PHBE PWM renamed PRINT HEAD BLOWER ENABLE
- net PRINT HEAD BLOWER ENABLE: now also U2.3 (1Y)
- net PRINT HEAD MODEL THEM renamed PRINT HEAD MODEL THERM
- net PRINT HEAD MODEL THERM: now also R5.2; no longer R8.2
- net PRINT HEAD SUPP THEM renamed PRINT HEAD SUPP THERM
- net T1 VSSA renamed VSSA0
- net VSSA0: now also J16.20 (Pin_20)
- net T2 VSSA renamed VSSA2
- net VSSA2: now also J16.24 (Pin_24)
- net VD CHAMBER HEATER ENABLE renamed 48v
- net 48v: now also J16.5 (Pin_5)
- new net: J6.1 (Pin_1), U3.7 (PA10)
- new net 120V ON: J5.16 (Pin_16), U1.3 (1Y)
- new net 48v RTN PWM: J16.3 (Pin_3), R1.1, R2.2, U1.1 (1~{OE}), U1.10 (3~{OE}), U1.13 (4~{OE}), U1.4 (2~{OE}), U2.1 (1~{OE}), U2.10 (3~{OE}), U2.13 (4~{OE}), U2.4 (2~{OE})
- new net I_SPR1: J14.7 (Pin_7), R14.2, U4.13 (PA12)
- new net I_SPR2: J14.6 (Pin_6), R17.2, U4.25 (PA19)
- new net LS 120V ON: J16.2 (Pin_2), U1.2 (1A)
- new net LS CHAMBER HEATER ENABLE: J16.8 (Pin_8), U1.12 (4A)
- new net LS EXTRUDER MODEL HEATER ENABLE: J16.14 (Pin_14), U2.9 (3A)
- new net LS EXTRUDER SUPPORT HEATER ENABLE: J16.12 (Pin_12), U2.5 (2A)
- new net LS PRINT HEAD BLOWER ENABLE: J16.10 (Pin_10), U2.2 (1A)
- new net SPR1: J14.3 (Pin_3), U4.1 (PA02)
- new net SPR2: J14.5 (Pin_5), U4.2 (PA03)
- new net SPR3: J14.4 (Pin_4), U4.21 (PA23)
- new net SPR4: J14.2 (Pin_2), U4.22 (PA22)
- new net SPR5: J14.8 (Pin_8), U4.26 (PA18)
- new net SPR6: J14.10 (Pin_10), U4.27 (PA17)
- new net SPR7: J14.12 (Pin_12), U4.28 (PA16)
- new net SPR8: J14.14 (Pin_14), U4.24 (PA20)
- new net VSSA1: J16.28 (Pin_28), R3.1
- no-connect marks 75 -> 82
Other:
- note added: "Duet 3 Header"
- note added: "Level Shifters"
- note added: "Spares Header"
- note added: "Term"
- note added: "Voltage Divider"
- note removed: "Duet 3 Primary"
- note removed: "Duet 3 Secondary"
- note removed: "Level Shifter"
- note removed: "Voltage Dividers"
- title: DUEPRINT3 - STRATASYS TO DUET 3 INTERFACE BOARD v1.0.0 -> DUEPRINT3 - STRATASYS TO DUET 3 INTERFACE BOARD v2.0.0
- moved on the sheet: C1, H1, H2, H3, H4, H5, J1, J11, J12, J13, J2, J3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
