File: DuePrint3 KiCad Project/DuePrint3.kicad_sch (KiCad schematic)
At the start: 41 parts, among them J1 EHT-110-01-S-D, J11 6P2C, J12 6P2C, J13 2.54Header-1x3-M, J14 Conn_02x07_Top_Bottom, J16 Conn_02x15_Odd_Even, J2 EHT-125-01-S-D, J3 MF3.0-1x2-436500215, J4 MF3.0-1x2-436500215, J5 EHT-125-01-S-D, J6 Conn_01x02, J8 MF3.0-1x2-436500215, U1 SN74AHCT125DR, U2 SN74AHCT125DR, U3 BLACKPILL, U4 SAMMY-C21

Commit message: Progress on v2.5.0
Parts:
- removed U3: BLACKPILL, DuePrint3-Lib:STM32 BLACKPILL, symbol DuePrint3:STM32F411_BLACKPILL
- added D1: 12V, LED_SMD:LED_0603_1608Metric_Pad1.05x0.95mm_HandSolder, symbol Device:LED
- added D2: 5V_SW, LED_SMD:LED_0603_1608Metric_Pad1.05x0.95mm_HandSolder, symbol Device:LED
- added D3: 5V, LED_SMD:LED_0603_1608Metric_Pad1.05x0.95mm_HandSolder, symbol Device:LED
- added J9: MF3.0-1x2-436500215, Connector_Molex:Molex_Micro-Fit_3.0_43650-0215_1x02_P3.00mm_Vertical, symbol Connector_Generic:Conn_01x02
- added R18: 10k, Resistor_SMD:R_0805_2012Metric_Pad1.20x1.40mm_HandSolder, symbol Device:R
- added R19, R20: 2K2, Resistor_SMD:R_0805_2012Metric_Pad1.20x1.40mm_HandSolder, symbol Device:R
- J4: value MF3.0-1x2-436500215 -> MF3.0-1x2-436500315; footprint Connector_Molex:Molex_Micro-Fit_3.0_43650-0215_1x02_P3.00mm_Vertical -> Connector_Molex:Molex_Micro-Fit_3.0_43650-0315_1x03_P3.00mm_Vertical; symbol Connector_Generic:Conn_01x02 -> Connector_Generic:Conn_01x03
- J6: value Conn_01x02 -> MF3.0-1x2-436500215; footprint Connector_PinHeader_2.54mm:PinHeader_2x01_P2.54mm_Vertical -> Connector_Molex:Molex_Micro-Fit_3.0_43650-0215_1x02_P3.00mm_Vertical
- U4: value SAMMY-C21 -> DP3EXB; footprint DuePrint3-Lib:SAMMY-C21 -> DuePrint3-Lib:DP3EXB; symbol DuePrint3:SAMMY-C21 -> DuePrint3:DP3EXB
Connections:
- net DIR is gone; now on net ENCODER CH B: U4.11 (PA25)
- net STEP is gone; now on net ENCODER CH A: U4.12 (PA24)
- net +12V: now also J4.3 (Pin_3), D1.2 (A); no longer J4.2 (Pin_2)
- net +5V: now also J6.2 (Pin_2), D3.2 (A), J9.2 (Pin_2); no longer U4.15 (V33)
- net 48v RTN PWM: now also D2.2 (A)
- net ARMATURE NEGATIVE: now also U4.28 (PA13)
- net ARMATURE POSITIVE: now also U4.27 (PA20)
- net GND: now also J4.2 (Pin_2), J6.1 (Pin_1), J9.1 (Pin_1), R18.1, R19.2, R20.2; no longer J4.1 (Pin_1), J6.2 (Pin_2)
- net Print Head Model Toggle SW: now also U4.30 (PB11); no longer U4.3 (PB08)
- net SPR6: no longer J14.10 (Pin_10), U4.27 (PA17)
- net SPR7: no longer J14.12 (Pin_12), U4.28 (PA16)
- new net: D1.1 (K), R18.2
- new net: D2.1 (K), R20.1
- new net: D3.1 (K), R19.1
- no-connect marks 82 -> 55
Other:
- note added: "DP3EXB MCU Module"
- note removed: "STM32 Extruder"
- note removed: "Sammy C21 MCU Module"
- moved on the sheet: J3, J8, R15, R17

Commit message: 4layer test
Parts:
- added J15: 2.54Header-1x3-M, Connector_PinHeader_2.54mm:PinHeader_1x03_P2.54mm_Vertical, symbol Connector_Generic:Conn_01x03
- added J90, J91: Conn_01x16_Socket, Connector_PinHeader_2.54mm:PinHeader_1x16_P2.54mm_Vertical, symbol Connector:Conn_01x16_Socket
- added J92, J93: Conn_01x02, symbol Connector_Generic:Conn_01x02
- D1: footprint LED_SMD:LED_0603_1608Metric_Pad1.05x0.95mm_HandSolder -> LED_SMD:LED_0805_2012Metric_Pad1.15x1.40mm_HandSolder; Part Number 150060BS75000 or equivalent Blue -> 150080BS75000
- D2: footprint LED_SMD:LED_0603_1608Metric_Pad1.05x0.95mm_HandSolder -> LED_SMD:LED_0805_2012Metric_Pad1.15x1.40mm_HandSolder; Part Number LTST-C191KGKT -> 150080VS75000
- D3: footprint LED_SMD:LED_0603_1608Metric_Pad1.05x0.95mm_HandSolder -> LED_SMD:LED_0805_2012Metric_Pad1.15x1.40mm_HandSolder; Part Number 150060AS75000 -> 150080AS75000
Connections:
- net ARMATURE NEGATIVE: now also U4.27 (PA20); no longer U4.28 (PA13)
- net ARMATURE POSITIVE: now also U4.28 (PA13); no longer U4.27 (PA20)
- net LS MOTOR ENABLE: now also J15.2 (Pin_2); no longer J16.6 (Pin_6)
- net SPR6: now also J14.10 (Pin_10), U4.9 (PA09)
- net SPR7: now also J14.12 (Pin_12), U4.10 (PA11)
- net MOTOR EN EXB: now reaches U4.4 (PB09)
- net MOTOR EN EXB: now also J15.1 (Pin_1)
- new net MOTOR EN MB: J15.3 (Pin_3), J16.6 (Pin_6)
- no-connect marks 55 -> 52

Commit message: Updating documentation for v2.5.0
Parts:
- C1, C2: Part Number (none) -> CL21B104KCFSFNE
- C3: Part Number (none) -> CL21B103KAANNNC
- J1: Part Number (none) -> EHT-110-01-S-D
- J11, J12: Part Number (none) -> SS-6466S-A-PG1
- J13, J15: Part Number (none) -> 61300311121
- J14: Part Number (none) -> B14B-PHDSS
- J16: Part Number (none) -> B30B-PHDSS
- J2, J5: Part Number (none) -> EHT-125-01-S-D
- J3, J6, J8, J9: Part Number (none) -> 436500215
- J4: Part Number (none) -> 436500315
- J90, J91: Part Number (none) -> 61301611821
- J92, J93: value Conn_01x02 -> 2 Pin Jumper; Part Number (none) -> QPC02SXGN-RC
- R1: Part Number (none) -> CRCW08053K74FKEA
- R10, R11, R12, R13, R14, R15, R17, R18: Part Number (none) -> CRCW080510K0FKEA
- R16: Part Number (none) -> CRCW0805120RFKEA
- R19, R20: Part Number xxRK73H1ETTP2201F -> CRCW08052K20FKEA
- R2: Part Number (none) -> CRCW080531K6FKEA
- R3, R4, R6: Part Number (none) -> CRCW08052K00FKEA
- R5, R7, R8: Part Number (none) -> CRCW08051K00FKEA
- R9: Part Number (none) -> ERJ-6ENF1003V
- U1, U2: Part Number (none) -> SN74AHCT125DR
- U4: Part Number (none) -> DP3EXB
