File: DuePrint3 KiCad Project/DuePrint3.kicad_pcb (KiCad board)
At the start: 2 copper layers, 208.2 x 43.6 mm, 42 parts, among them J1 EHT-110-01-S-D, J11 6P2C, J12 6P2C, J13 2.54Header-1x3-M, J14 Conn_02x07_Top_Bottom, J16 Conn_02x15_Odd_Even, J2 EHT-125-01-S-D, J3 MF3.0-1x2-436500215, J4 MF3.0-1x2-436500215, J5 EHT-125-01-S-D, J6 Conn_01x02, J8 MF3.0-1x2-436500215, U1 SN74AHCT125DR, U2 SN74AHCT125DR, U3 BLACKPILL, U4 SAMMY-C21

Commit message: Progress on v2.5.0
Parts:
- removed REF**: OSHW-Logo2_7.3x6mm_SilkScreen, Symbol:OSHW-Logo2_7.3x6mm_SilkScreen
- removed U3: BLACKPILL, DuePrint3-Lib:STM32 BLACKPILL
- added D1: 12V, LED_SMD:LED_0603_1608Metric_Pad1.05x0.95mm_HandSolder, F.Cu at (63.1, 40.5)
- added D2: 5V_SW, LED_SMD:LED_0603_1608Metric_Pad1.05x0.95mm_HandSolder, F.Cu at (63.1, 50.0)
- added D3: 5V, LED_SMD:LED_0603_1608Metric_Pad1.05x0.95mm_HandSolder, F.Cu at (63.1, 44.8)
- added J9: MF3.0-1x2-436500215, Connector_Molex:Molex_Micro-Fit_3.0_43650-0215_1x02_P3.00mm_Vertical, F.Cu at (240.0, 53.4)
- added R18: 10k, Resistor_SMD:R_0805_2012Metric_Pad1.20x1.40mm_HandSolder, F.Cu at (63.1, 38.3)
- added R19: 2K2, Resistor_SMD:R_0805_2012Metric_Pad1.20x1.40mm_HandSolder, F.Cu at (63.1, 42.6)
- added R20: 2K2, Resistor_SMD:R_0805_2012Metric_Pad1.20x1.40mm_HandSolder, F.Cu at (63.1, 47.8)
- J4: value MF3.0-1x2-436500215 -> MF3.0-1x2-436500315; footprint Connector_Molex:Molex_Micro-Fit_3.0_43650-0215_1x02_P3.00mm_Vertical -> Connector_Molex:Molex_Micro-Fit_3.0_43650-0315_1x03_P3.00mm_Vertical
- J6: value Conn_01x02 -> MF3.0-1x2-436500215; footprint Connector_PinHeader_2.54mm:PinHeader_2x01_P2.54mm_Vertical -> Connector_Molex:Molex_Micro-Fit_3.0_43650-0215_1x02_P3.00mm_Vertical
- U4: value SAMMY-C21 -> DP3EXB; footprint DuePrint3-Lib:SAMMY-C21 -> DuePrint3-Lib:DP3EXB
- moved J6 34.1 mm to (227.6, 53.2)
- moved R15 27.1 mm to (120.2, 56.1), turned to -90 degrees
- moved J4 3.00 mm to (212.4, 66.0)
Connections:
- J14 pad 10: SPR6 -> unconnected-(J14-Pin_10-Pad10)
- J14 pad 12: SPR7 -> unconnected-(J14-Pin_12-Pad12)
- J4 pad 1: GND -> unconnected-(J4-Pin_1-Pad1)
- J4 pad 2: +12V -> GND
- J6 pad 1: Net-(J6-Pin_1) -> GND
- J6 pad 2: GND -> +5V
- U4 pad 11: DIR -> ENCODER CH B
- U4 pad 12: STEP -> ENCODER CH A
- U4 pad 15: +5V -> unconnected-(U4-V33-Pad15)
- U4 pad 27: SPR6 -> ARMATURE POSITIVE
- U4 pad 28: SPR7 -> ARMATURE NEGATIVE
- U4 pad 3: Print Head Model Toggle SW -> unconnected-(U4-PB08-Pad3)
- U4 pad 30: unconnected-(U4-CAN1_H-Pad30) -> Print Head Model Toggle SW
Routing:
- net DIR: track 159.2 -> 0.00 mm
- net STEP: track 151.8 -> 0.00 mm
- net ENCODER CH B: track 45.0 -> 167.2 mm, vias 0 -> 2
- net ENCODER CH A: track 46.2 -> 164.7 mm, vias 0 -> 2
- net ARMATURE POSITIVE: track 28.5 -> 129.5 mm, vias 0 -> 1
- net ARMATURE NEGATIVE: track 29.4 -> 127.6 mm, vias 0 -> 1
- net SPR7: track 38.8 -> 0.00 mm
- net SPR6: track 37.2 -> 0.00 mm
- net Print Head Model Toggle SW: track 31.2 -> 65.2 mm
- net +12V: track 225.4 -> 245.2 mm, vias 0 -> 1
- net 48v RTN PWM: track 68.2 -> 87.1 mm, vias 8 -> 10
- net Net-(J6-Pin_1): track 14.5 -> 0.00 mm
- net +5V: track 35.2 -> 39.9 mm
- net Net-(D3-K): track 0.00 -> 2.25 mm
- net Net-(D2-K): track 0.00 -> 2.25 mm
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Other:
- board text added: "+5V"
- board text added: "DP3EXB"
- board text added: "v2.5.0"
- board text removed: "SAMMY-C21"
- board text removed: "VCC"
- board text removed: "v2.0.0"

Commit message: 4layer test
Parts:
- added J15: 2.54Header-1x3-M, Connector_PinHeader_2.54mm:PinHeader_1x03_P2.54mm_Vertical, F.Cu at (74.4, 42.0)
- added REF**: OSHW-Logo2_7.3x6mm_SilkScreen, Symbol:OSHW-Logo2_7.3x6mm_SilkScreen, F.Cu at (105.7, 63.4)
- C1, C2, R10, R11, R12, R13, R14, R15, R17, U1, U2: moved to F.Cu
- D1, D2, D3: footprint LED_SMD:LED_0603_1608Metric_Pad1.05x0.95mm_HandSolder -> LED_SMD:LED_0805_2012Metric_Pad1.15x1.40mm_HandSolder
- moved R14 13.0 mm to (123.7, 43.3), turned to -90 degrees
- moved R10 12.9 mm to (134.4, 43.3), turned to -90 degrees
- moved R11 12.9 mm to (138.0, 43.3), turned to -90 degrees
- moved R12 12.9 mm to (141.6, 43.3), turned to 90 degrees
- moved R13 12.9 mm to (145.2, 43.3), turned to 90 degrees
- moved R17 12.9 mm to (130.8, 43.3)
- moved R15 12.8 mm to (120.2, 43.3)
- moved R1 9.74 mm to (102.9, 52.9), turned to 0 degrees
- moved C1 9.50 mm to (95.4, 53.9), turned to 0 degrees
- moved C2 7.20 mm to (80.4, 52.1), turned to 180 degrees
- moved R2 6.83 mm to (102.9, 55.4), turned to 180 degrees
- moved U2 4.75 mm to (87.1, 48.1)
- moved U1 4.53 mm to (96.8, 48.2)
- moved J9 3.38 mm to (243.4, 53.5), turned to 180 degrees
- moved J6 3.32 mm to (230.9, 53.5), turned to 180 degrees
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Connections:
- J14 pad 10: unconnected-(J14-Pin_10-Pad10) -> SPR6
- J14 pad 12: unconnected-(J14-Pin_12-Pad12) -> SPR7
- J16 pad 6: LS MOTOR ENABLE -> MOTOR EN MB
- U4 pad 10: unconnected-(U4-PA11-Pad10) -> SPR7
- U4 pad 27: ARMATURE POSITIVE -> ARMATURE NEGATIVE
- U4 pad 28: ARMATURE NEGATIVE -> ARMATURE POSITIVE
- U4 pad 4: unconnected-(U4-PB09-Pad4) -> MOTOR EN EXB
- U4 pad 9: unconnected-(U4-PA09-Pad9) -> SPR6
Routing:
- net MOTOR EN EXB: track 0.00 -> 75.0 mm, vias 0 -> 1
- net SPR7: track 0.00 -> 35.3 mm, vias 0 -> 1
- net SPR6: track 0.00 -> 32.3 mm, vias 0 -> 1
- net MOTOR EN MB: track 0.00 -> 29.2 mm, vias 0 -> 1
- net POWER ON: track 39.4 -> 17.8 mm, vias 1 -> 0
- net +5V: track 39.9 -> 21.8 mm, vias 4 -> 7
- net Print Head Model Toggle SW: track 65.2 -> 79.7 mm
- net I_SPR2: track 42.6 -> 56.0 mm, vias 0 -> 1
- net LS MOTOR ENABLE: track 7.16 -> 20.5 mm, vias 0 -> 1
- net EXTRUDER SUPPORT HEATER ENABLE: track 39.8 -> 27.7 mm, vias 4 -> 1
- net MOTOR ENABLE: track 129.8 -> 118.4 mm, vias 1 -> 0
- net EXTRUDER MODEL HEATER ENABLE: track 42.2 -> 32.1 mm, vias 3 -> 2
- net LS EXTRUDER MODEL HEATER ENABLE: track 8.36 -> 17.1 mm, vias 0 -> 1
- net LS EXTRUDER SUPPORT HEATER ENABLE: track 7.90 -> 16.6 mm, vias 0 -> 1
- net 120V ON: track 29.0 -> 21.3 mm, vias 1 -> 0
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- added copper zone on In2.Cu, net +5V
- added copper zone on In1.Cu, net GND
- removed copper zone on F.Cu, net +5V
- removed copper zone on B.Cu, net GND
Other:
- copper layers 2 -> 4
- board text added: "EXB"
- board text added: "MAIN_BRD"

Commit message: Updating documentation for v2.5.0
Routing:
- net +5V: track 21.8 -> 5.27 mm, vias 7 -> 0
- net ENCODER CH A: track 164.7 -> 163.7 mm, vias 0 -> 4
- net CHAMBER TEMP ALARM: track 150.2 -> 151.0 mm, vias 1 -> 5
- net MOTOR EN EXB: track 75.0 -> 75.6 mm
- net LS EXTRUDER MODEL HEATER ENABLE: track 17.1 -> 16.5 mm
- net LS POWER ON: track 17.2 -> 16.6 mm
- net POWER I/O: track 81.3 -> 81.7 mm, vias 0 -> 4
- net ARMATURE POSITIVE: track 132.3 -> 132.5 mm, vias 1 -> 3
- net ENCODER CH B: vias 0 -> 4
- net +12V: vias 3 -> 9
- net PRINT HEAD TEMP ALARM: vias 0 -> 2
- net ARMATURE NEGATIVE: vias 1 -> 3
- net Print Head Model Toggle SW: vias 2 -> 4
- added copper zone on F.Cu, net +5V
- added copper zone on B.Cu, net GND
- removed copper zone on In2.Cu, net +5V
- removed copper zone on In1.Cu, net GND
Other:
- copper layers 4 -> 2
